Commit message: Fix torque derating bug, recalibrate stand height, retune actuator gains
- build_mjcf.py: override actuated-joint effort limit to 2.5 N·m (was
  silently inherited as 1.0 N·m from the Onshape URDF export, capping
  every servo at a third of its intended output).
- postprocess.py: recalibrate STAND_HEIGHT from 0.2061 to 0.2030 using
  foot mesh AABB corners, so both feet register contact at the standing
  pose instead of floating 1-3mm above the floor. Retune actuator gains
  from kp=5.0/kv=0.2 to kp=40.0/kv=10.0 after direct testing showed the
  old gains produced unrealistic no-load speeds (2.4-3.4x the ST3215
  spec) and excessive gravity-loaded steady-state error; the new gains
  bring both within target while keeping overshoot at 0%.
- pyproject.toml: pin mujoco>=3.10,<4 and requires-python>=3.10 to match
  the installed/verified version and the mujoco package's own metadata.
- Regenerated biped.xml, biped_no_jetson.xml, biped_raw.xml, and the
  intermediate URDF from the updated pipeline.

File: models/urdf/biped_for_mujoco.urdf (robot description, URDF)
Before this commit: robot assembly_simple, 35 links, 34 joints
Joints:
- joint hip_pitch_l: limit lower=-1.39626 upper=1.39626 effort=1 velocity=1 -> lower=-1.39626 upper=1.39626 effort=2.5 velocity=1
- joint hip_pitch_r: limit lower=-1.39626 upper=1.39626 effort=1 velocity=1 -> lower=-1.39626 upper=1.39626 effort=2.5 velocity=1
- joint hip_roll_l: limit lower=-2.26893 upper=0.0872665 effort=1 velocity=1 -> lower=-2.26893 upper=0.0872665 effort=2.5 velocity=1
- joint hip_roll_r: limit lower=-0.0872665 upper=2.26893 effort=1 velocity=1 -> lower=-0.0872665 upper=2.26893 effort=2.5 velocity=1
- joint knee_l: limit lower=-1.39626 upper=1.39626 effort=1 velocity=1 -> lower=-1.39626 upper=1.39626 effort=2.5 velocity=1
- joint knee_r: limit lower=-1.39626 upper=1.39626 effort=1 velocity=1 -> lower=-1.39626 upper=1.39626 effort=2.5 velocity=1

Commit message: Phase 6.A: mjlab entity config + fix keyframe/forcerange bugs; rename actuators to match hardware firmware
- Fix Phase 6.A bugs: actuator_forcerange 2D-array indexing, mjOBJ_KEYFRAME -> mjOBJ_KEY
- Rename actuated joints to match motor controller/joint encoder firmware naming:
  hip_pitch->knee, knee->ankle (hip_roll unchanged)
- Rename passive hardstop joint ankle->foot to avoid colliding with the
  newly-renamed actuated ankle_l/r
- Regenerate biped.xml, biped_no_jetson.xml, biped_warp.xml with new joint names
- Rename test_ankles_collision.py -> test_foot_collision.py, TestKneePendulum ->
  TestAnklePendulum to match
- Update all prose references across tests, README, and docs

File: models/urdf/biped_for_mujoco.urdf (robot description, URDF)
Before this commit: robot assembly_simple, 35 links, 34 joints
Joints:
- removed joint hip_pitch_l
- removed joint hip_pitch_r
- added joint foot_l: type revolute, parent tube_4, child foot_1, origin xyz=0 0.025 2.77556e-17 rpy=0.528547 5.55112e-17 -1.5708, axis 1 -0 -0, limit lower=-0.314159 upper=0.296706 effort=0 velocity=20
- added joint foot_r: type revolute, parent tube_2, child foot, origin xyz=-3.25261e-18 0.025 -2.77556e-17 rpy=0.5321 7.27196e-15 -1.5708, axis 1 -0 -0, limit lower=-0.314159 upper=0.296706 effort=0 velocity=20
- joint ankle_l: axis 1 -0 -0 -> 0 -1 0; child foot_1 -> tibia_2; limit lower=-0.314159 upper=0.296706 effort=0 velocity=20 -> lower=-1.39626 upper=1.39626 effort=2.5 velocity=1; origin xyz=0 0.025 2.77556e-17 rpy=0.528547 5.55112e-17 -1.5708 -> xyz=-0.0338 -0.03575 -0.0113 rpy=-5.26172e-17 -5.37322e-14 -3.14159; parent tube_4 -> motor
- joint ankle_r: axis 1 -0 -0 -> 0 1 0; child foot -> tibia_1; limit lower=-0.314159 upper=0.296706 effort=0 velocity=20 -> lower=-1.39626 upper=1.39626 effort=2.5 velocity=1; origin xyz=-3.25261e-18 0.025 -2.77556e-17 rpy=0.5321 7.27196e-15 -1.5708 -> xyz=-0.03 -0.00075 -0.0113 rpy=3.14159 2.49218e-15 3.14159; parent tube_2 -> motor_2
- joint knee_l: child tibia_2 -> hip_joint_a; origin xyz=-0.0338 -0.03575 -0.0113 rpy=-5.26172e-17 -5.37322e-14 -3.14159 -> xyz=-0.0338 0.00075 0.0113 rpy=0 1.5708 8.11363e-17; parent motor -> motor_3
- joint knee_r: axis 0 1 0 -> -0 -1 -0; child tibia_1 -> motor_1; origin xyz=-0.03 -0.00075 -0.0113 rpy=3.14159 2.49218e-15 3.14159 -> xyz=0.00314735 -0.002 0.016 rpy=0 -1.5708 3.14159; parent motor_2 -> hip_joint_b_2
